Commit message: add process_image impl. Not working though.

File: src/my_robot/urdf/my_robot.xacro (robot description, xacro)
@@ -81,5 +81,4 @@
   </link>
   <link name='right_wheel'>
-  <!-- left wheel -->
       <pose>1 1 1 0 0 0</pose>
       <inertial>
@@ -115,5 +114,5 @@
   <joint name="right_wheel_hinge" type="continuous">
     <origin xyz="0 -0.15 0" rpy="0 0 0" />
-    <axis xyz="0 -1 0" rpy="0 0 0"/>
+    <axis xyz="0 1 0" rpy="0 0 0"/>
     <limit effort="10000" velocity="1000"/>
     <dynamics damping="1.0" friction="1.0"/>

Commit message: working on changing the robot design

File: src/my_robot/urdf/my_robot.xacro (robot description, xacro)
@@ -8,5 +8,4 @@
   </joint>
   <link name='chassis'>
-    <pose>0 0 0.1 0 0 0</pose>
     <inertial>
       <mass value="15.0"/>
@@ -21,5 +20,5 @@
       <origin xyz="0 0 0" rpy=" 0 0 0"/>
       <geometry>
-        <box size=".4 .2 .1"/>
+        <box size=".5 .3 .1"/>
       </geometry>
     </collision>
@@ -27,45 +26,31 @@
       <origin xyz="0 0 0" rpy=" 0 0 0"/>
       <geometry>
-        <box size=".4 .2 .1"/>
-      </geometry>
-    </visual>
-    <collision name='back_caster_collision'>
-      <origin xyz="-0.15 0 -0.05" rpy=" 0 0 0"/>
-      <geometry>
-        <sphere radius="0.0499"/>
-      </geometry>
-    </collision>
-    <visual name='back_caster_visual'>
-      <origin xyz="-0.15 0 -0.05" rpy=" 0 0 0"/>
-      <geometry>
-        <sphere radius="0.05"/>
+        <box size=".5 .3 .1"/>
       </geometry>
     </visual>
     <collision name='front_caster_collision'>
-      <origin xyz="0.15 0 -0.05" rpy=" 0 0 0"/>
+      <origin xyz="0.13 0 -0.05" rpy=" 0 0 0"/>
       <geometry>
-        <sphere radius="0.0499"/>
+        <sphere radius="0.08"/>
       </geometry>
     </collision>
     <visual name='front_caster_visual'>
-      <origin xyz="0.15 0 -0.05" rpy=" 0 0 0"/>
+      <origin xyz="0.13 0 -0.05" rpy=" 0 0 0"/>
       <geometry>
-        <sphere radius="0.05"/>
+        <sphere radius="0.08"/>
       </geometry>
     </visual>
   </link>
   <link name='left_wheel'>
-  <!-- left wheel -->
-      <pose>1 1 1 0 0 0</pose>
-      <inertial>
-      	<mass value="5.0"/>
-      	<origin xyz="0.0 0 0" rpy=" 0 0 0"/>
-      	<inertia
-          ixx="0.1" ixy="0" ixz="0"
-          iyy="0.1" iyz="0"
-          izz="0.1"
-      	/>
-      </inertial>
-    <collision name='collision'>
+    <inertial>
+      <mass value="5.0"/>
+      <origin xyz="0.0 0 0" rpy=" 0 0 0"/>
+      <inertia
+        ixx="0.1" ixy="0" ixz="0"
+        iyy="0.1" iyz="0"
+        izz="0.1"
+      />
+    </inertial>
+    <collision name='left_wheel_collision'>
       <origin xyz="0 0 0" rpy=" 0 1.5707 1.5707"/>
       <geometry>
@@ -80,16 +65,23 @@
     </visual>
   </link>
+  <joint name="left_wheel_hinge" type="continuous">
+    <origin xyz="-0.15 -0.18 -0.04" rpy="0 0 0" />
+    <axis xyz="0 1 0" rpy="0 0 0"/>
+    <limit effort="10000" velocity="1000"/>
+    <dynamics damping="1.0" friction="1.0"/>
+    <parent link="chassis"/>
+    <child link="left_wheel" />
+  </joint>
   <link name='right_wheel'>
-      <pose>1 1 1 0 0 0</pose>
-      <inertial>
-      	<mass value="5.0"/>
-      	<origin xyz="0.0 0 0" rpy=" 0 0 0"/>
-      	<inertia
-          ixx="0.1" ixy="0" ixz="0"
-          iyy="0.1" iyz="0"
-          izz="0.1"
-      	/>
-      </inertial>
-    <collision name='collision'>
+    <inertial>
+      <mass value="5.0"/>
+      <origin xyz="0.0 0 0" rpy=" 0 0 0"/>
+      <inertia
+        ixx="0.1" ixy="0" ixz="0"
+        iyy="0.1" iyz="0"
+        izz="0.1"
+      />
+    </inertial>
+    <collision name='right_wheel_collision'>
       <origin xyz="0 0 0" rpy=" 0 1.5707 1.5707"/>
       <geometry>
@@ -104,14 +96,6 @@
     </visual>
   </link>
-  <joint name="left_wheel_hinge" type="continuous">
-    <origin xyz="0 0.15 0" rpy="0 0 0" />
-    <axis xyz="0 1 0" rpy="0 0 0"/>
-    <limit effort="10000" velocity="1000"/>
-    <dynamics damping="1.0" friction="1.0"/>
-    <parent link="chassis"/>
-    <child link="left_wheel" />
-  </joint>
   <joint name="right_wheel_hinge" type="continuous">
-    <origin xyz="0 -0.15 0" rpy="0 0 0" />
+    <origin xyz="-0.15 0.18 -0.04" rpy="0 0 0" />
     <axis xyz="0 1 0" rpy="0 0 0"/>
     <limit effort="10000" velocity="1000"/>
@@ -120,6 +104,15 @@
     <child link="right_wheel" />
   </joint>
+<gazebo reference="chassis">
+    <material>Gazebo/SkyBlue</material>
+</gazebo>
+<gazebo reference="left_wheel">
+    <material>Gazebo/Indigo</material>
+</gazebo>
+<gazebo reference="right_wheel">
+    <material>Gazebo/Indigo</material>
+</gazebo>
   <link name="camera">
-      <origin xyz="0 0 0" rpy="0 0 0" />
+    <origin xyz="0 0 0" rpy="0 0 0" />
     <inertial>
       <mass value="0.1"/>
@@ -142,5 +135,5 @@
   <joint name="camera_joint" type="fixed">
     <axis xyz="0 1 0" rpy="0 0 0"/>
-    <origin xyz="0.2 0 0" rpy="0 0 0" />
+    <origin xyz="0.25 0 0" rpy="0 0 0" />
     <parent link="chassis"/>
     <child link="camera" />
@@ -168,19 +161,10 @@
   <joint name="hokuyo_joint" type="fixed">
     <axis xyz="0 1 0" rpy="0 0 0"/>
-    <origin xyz="0.15 0 .1" rpy="0 0 0" />
+    <origin xyz="0 0 .1" rpy="0 0 0" />
     <parent link="chassis"/>
     <child link="hokuyo" />
   </joint>
-<gazebo reference="left_wheel">
+<gazebo reference="camera">
     <material>Gazebo/Green</material>
 </gazebo>
-<gazebo reference="right_wheel">
-    <material>Gazebo/Green</material>
-</gazebo>
-<gazebo reference="chassis">
-    <material>Gazebo/Blue</material>
-</gazebo>
-<gazebo reference="camera">
-    <material>Gazebo/Red</material>
-</gazebo>
 </robot>

Commit message: Added sensor base

File: src/my_robot/urdf/my_robot.xacro (robot description, xacro)
@@ -20,5 +20,5 @@
       <origin xyz="0 0 0" rpy=" 0 0 0"/>
       <geometry>
-        <box size=".5 .3 .1"/>
+        <box size=".5 .2 .1"/>
       </geometry>
     </collision>
@@ -26,17 +26,29 @@
       <origin xyz="0 0 0" rpy=" 0 0 0"/>
       <geometry>
-        <box size=".5 .3 .1"/>
+        <box size=".5 .2 .1"/>
       </geometry>
     </visual>
     <collision name='front_caster_collision'>
-      <origin xyz="0.13 0 -0.05" rpy=" 0 0 0"/>
+      <origin xyz="-0.15 0 -0.05" rpy=" 0 0 0"/>
       <geometry>
-        <sphere radius="0.08"/>
+        <sphere radius="0.07"/>
       </geometry>
     </collision>
     <visual name='front_caster_visual'>
-      <origin xyz="0.13 0 -0.05" rpy=" 0 0 0"/>
+      <origin xyz="-0.15 0 -0.05" rpy=" 0 0 0"/>
       <geometry>
-        <sphere radius="0.08"/>
+        <sphere radius="0.07"/>
+      </geometry>
+    </visual>
+    <collision name='back_caster_collision'>
+      <origin xyz="0.15 0 -0.05" rpy=" 0 0 0"/>
+      <geometry>
+        <sphere radius="0.07"/>
+      </geometry>
+    </collision>
+    <visual name='back_caster_visual'>
+      <origin xyz="0.15 0 -0.05" rpy=" 0 0 0"/>
+      <geometry>
+        <sphere radius="0.07"/>
       </geometry>
     </visual>
@@ -55,5 +67,5 @@
       <origin xyz="0 0 0" rpy=" 0 1.5707 1.5707"/>
       <geometry>
-        <cylinder radius="0.1" length="0.05"/>
+        <cylinder radius="0.12" length="0.05"/>
       </geometry>
     </collision>
@@ -61,10 +73,10 @@
       <origin xyz="0 0 0" rpy=" 0 1.5707 1.5707"/>
       <geometry>
-        <cylinder radius="0.1" length="0.05"/>
+        <cylinder radius="0.12" length="0.05"/>
       </geometry>
     </visual>
   </link>
   <joint name="left_wheel_hinge" type="continuous">
-    <origin xyz="-0.15 -0.18 -0.04" rpy="0 0 0" />
+    <origin xyz="0 -0.13 0" rpy="0 0 0" />
     <axis xyz="0 1 0" rpy="0 0 0"/>
     <limit effort="10000" velocity="1000"/>
@@ -86,5 +98,5 @@
       <origin xyz="0 0 0" rpy=" 0 1.5707 1.5707"/>
       <geometry>
-        <cylinder radius="0.1" length="0.05"/>
+        <cylinder radius="0.12" length="0.05"/>
       </geometry>
     </collision>
@@ -92,10 +104,10 @@
       <origin xyz="0 0 0" rpy=" 0 1.5707 1.5707"/>
       <geometry>
-        <cylinder radius="0.1" length="0.05"/>
+        <cylinder radius="0.12" length="0.05"/>
       </geometry>
     </visual>
   </link>
   <joint name="right_wheel_hinge" type="continuous">
-    <origin xyz="-0.15 0.18 -0.04" rpy="0 0 0" />
+    <origin xyz="0 0.13 0" rpy="0 0 0" />
     <axis xyz="0 1 0" rpy="0 0 0"/>
     <limit effort="10000" velocity="1000"/>
@@ -105,11 +117,11 @@
   </joint>
 <gazebo reference="chassis">
-    <material>Gazebo/SkyBlue</material>
+    <material>Gazebo/BlueGlow</material>
 </gazebo>
 <gazebo reference="left_wheel">
-    <material>Gazebo/Indigo</material>
+    <material>Gazebo/PurpleGlow</material>
 </gazebo>
 <gazebo reference="right_wheel">
-    <material>Gazebo/Indigo</material>
+    <material>Gazebo/PurpleGlow</material>
 </gazebo>
   <link name="camera">
@@ -141,6 +153,18 @@
   <link name="hokuyo">
      <origin xyz="0 0 0" rpy="0 0 0" />
+    <collision name="base-collision">
+      <origin xyz="0 0 0.06" rpy=" 0 0 0"/>
+      <geometry>
+        <box size=".12 .12 .02"/>
+      </geometry>
+    </collision>
+    <visual name="base-visual">
+      <origin xyz="0 0 0.06" rpy=" 0 0 0"/>
+      <geometry>
+        <box size=".12 .12 .02"/>
+      </geometry>
+    </visual>
     <collision>
-      <origin xyz="0 0 0" rpy=" 0 0 0"/>
+      <origin xyz="0 0 .1" rpy=" 0 0 0"/>
       <geometry>
         <box size=".1 .1 .1"/>
@@ -148,5 +172,5 @@
     </collision>
     <visual>
-      <origin xyz="0 0 0" rpy=" 0 0 0"/>
+      <origin xyz="0 0 .1" rpy=" 0 0 0"/>
       <geometry>
         <mesh filename="package://my_robot/meshes/hokuyo.dae"/>
@@ -161,10 +185,10 @@
   <joint name="hokuyo_joint" type="fixed">
     <axis xyz="0 1 0" rpy="0 0 0"/>
-    <origin xyz="0 0 .1" rpy="0 0 0" />
+    <origin xyz="0.15 0 0.01" rpy="0 0 0" />
     <parent link="chassis"/>
     <child link="hokuyo" />
   </joint>
 <gazebo reference="camera">
-    <material>Gazebo/Green</material>
+    <material>Gazebo/Orange</material>
 </gazebo>
 </robot>
